File: RP2040-DebugProbe.kicad_sch (KiCad schematic)
At the start: 70 parts, among them J1 CONN_MCU_JTAG, J10 CONN_USB, J2 CONN_MCU_UART, J3 CONN_DBG_COMB, J4 CONN_3V3_JUMPER, J7 CONN_DBG_JTAG, SW1 BOOTSEL, U1 W25Q128JVS, U2 RP2040, U3 74AUP1T17, U4 W25Q128JVEIQ, U5 AMS1117-3.3, U6 74AUP1T17, Y1 12MHz

Commit message: tinyprogrammer
Parts:
- removed C1, C5: 2.2uF, Capacitor_SMD:C_0603_1608Metric, symbol Device:C_Small
- removed C12, C13: 100nF, Capacitor_SMD:C_0402_1005Metric, symbol Device:C_Small
- removed C21: 4.7nF 1kV, Capacitor_SMD:C_1206_3216Metric, symbol Device:C_Small
- removed FB2: 100@100MHz, Inductor_SMD:L_0805_2012Metric, symbol Device:FerriteBead_Small
- removed H1, H2, H3, H4: MountingHole_Pad, MountingHole:MountingHole_2.5mm_Pad_Via, symbol Mechanical:MountingHole_Pad
- removed J1: CONN_MCU_JTAG, Connector_PinHeader_1.27mm:PinHeader_2x05_P1.27mm_Vertical, symbol Connector:Conn_ARM_JTAG_SWD_10
- removed J2: CONN_MCU_UART, Connector_PinHeader_2.54mm:PinHeader_1x03_P2.54mm_Vertical, symbol Connector_Generic:Conn_01x03
- removed J3: CONN_DBG_COMB, Connector_PinHeader_2.54mm:PinHeader_1x08_P2.54mm_Vertical, symbol Connector_Generic:Conn_01x08
- removed J4: CONN_3V3_JUMPER, Connector_PinHeader_2.54mm:PinHeader_1x02_P2.54mm_Vertical, symbol Connector_Generic:Conn_01x02
- removed R20, R21, R22, R23: 100R, Resistor_SMD:R_0402_1005Metric, symbol Device:R_Small
- removed R8: 10k, Resistor_SMD:R_0402_1005Metric, symbol Device:R_Small
- removed SW1: BOOTSEL, PCM_4ms_Switch:Button_Tact_Sqkg, symbol Switch:SW_Push_Dual
- removed U1: W25Q128JVS, Package_SO:SOIC-8_5.23x5.23mm_P1.27mm, symbol Memory_Flash:W25Q128JVS
- removed U3, U6: 74AUP1T17, Package_TO_SOT_SMD:SOT-353_SC-70-5, symbol SN74AUP1T17DCKR:SN74AUP1T17DCKR
- removed U5: AMS1117-3.3, Package_TO_SOT_SMD:SOT-223-3_TabPin2, symbol Regulator_Linear:AMS1117-3.3
- added R24, R25: 27R, Resistor_SMD:R_0402_1005Metric, symbol Device:R_Small
- added TP10, TP11, TP13, TP4, TP5, TP6, TP7, TP8, TP9: TestPoint, TestPoint:TestPoint_Pad_D1.0mm, symbol Connector:TestPoint
- added U1: AP2112K-3.3, Package_TO_SOT_SMD:SOT-23-5, symbol Regulator_Linear:AP2112K-3.3
- added U3, U6: 74AUP1T17GWH, JLCPCB:TSSOP-5_L2.1-W1.3-P0.65-LS2.2-BR, symbol JLCPCB:74AUP1T17GWH
- added U5, U8: TS-1089S-02526, JLCPCB:SW-SMD_4P-L4.2-W3.3-P2.15-LS5.1, symbol JLCPCB:TS-1089S-02526
- C14, C15: value 10uF -> 22uF
- C19, C20: value 12pF -> 15pF
- J10: footprint Connector_USB:USB_C_Receptacle_HRO_TYPE-C-31-M-12 -> JLCPCB:USB-C-SMD_TYPE-C-6PIN-2MD-073; symbol Connector:USB_C_Receptacle_USB2.0 -> JLCPCB:TYPE-C_16PIN_2MD(073); LCSC (none) -> C2765186
- R12: value 1M -> 1K; footprint Resistor_SMD:R_0603_1608Metric -> Resistor_SMD:R_0402_1005Metric
- R19: value 100R -> 10k
- U4: value W25Q128JVEIQ -> W25Q64JVEIQ; footprint Package_SON:WSON-8-1EP_6x5mm_P1.27mm_EP3.4x4.3mm -> JLCPCB:USON-8_L4.0-W3.0-P0.80-BL_WINBOND_UU; symbol Memory_Flash:W25Q32JVZP -> JLCPCB:W25Q64JWUUIQ; LCSC (none) -> C6604692
- U7: renamed from J7; value CONN_DBG_JTAG -> HX_JN1_27-2X5_TP_H4_9; footprint Connector_PinHeader_1.27mm:PinHeader_2x05_P1.27mm_Vertical -> JLCPCB:IDC-SMD_10P-P1.27-3220-10-0300-00; symbol Connector:Conn_ARM_JTAG_SWD_10 -> JLCPCB:HX_JN1_27-2X5_TP_H4_9; LCSC (none) -> C42372555
- Y1: footprint Crystal:Crystal_SMD_3225-4Pin_3.2x2.5mm -> JLCPCB:CRYSTAL-SMD_4P-L3.2-W2.5-BL; symbol Device:Crystal_GND24_Small -> JLCPCB:ABM8-272-T3_C20625731; LCSC (none) -> C20625731
Connections:
- net MCU_RESET is gone; now on net RESET: U2.26 (RUN)
- net TARGET_3V3 is gone; now on net +5V: U7.1
- net +1V1: now also TP13.1
- net +3V3: now also R19.1, TP5.1, U1.5 (VOUT), U3.5 (VCC), U6.5 (VCC)
- net +5V: now also D3.4 (VCC), J10.11 (VBUS), J10.2 (VBUS), TP4.1, U1.1 (VIN), U1.3 (EN)
- net DBG_DIO_BUF: now also U6.4 (Y)
- net GND: now also D3.1 (GND), J10.1 (GND), J10.12 (GND), J10.13 (SHELL), J10.14 (SHELL), U4.10 (EP), U7.7, U1.2 (GND), U3.1 (NC), U3.3 (GND), U5.3, U5.4, U6.1 (NC), U6.3 (GND), U8.3, U8.4; no longer J10.A1 (GND), J10.A12 (GND), J10.B1 (GND), J10.B12 (GND), R12.2, R7.2
- net QSPI_SS: now also R7.1
- net TARGET_RX: now also U7.8
- net TARGET_TX: now also U7.6
- net UART_RX_BUF: now also U3.4 (Y)
- net USB_DN: now also R25.1; no longer D3.3 (I/O2), J10.A7 (D-), J10.B7 (D-)
- net USB_DP: now also R24.1; no longer D3.2 (I/O1), J10.A6 (D+), J10.B6 (D+)
- net XIN: now also Y1.1; no longer Y1.3
- net XOUT: now also R12.1; no longer C20.1, Y1.1
- net at R13.2: now also U6.2 (A)
- net RLED_RX: now reaches D1.2 (A), R1.2
- net at R9.2: now also U3.2 (A)
- net RLED_ACT: now reaches D5.2 (A), R3.2
- net RLED_CON: now reaches D6.2 (A), R4.2
- net CC1: now reaches R10.1
- net CC1: now also J10.4 (CC1); no longer J10.A5 (CC1)
- net CC2: now reaches R11.1
- net CC2: now also J10.10 (CC2); no longer J10.B5 (CC2)
- net RLED_TX: now reaches D4.2 (A), R2.2
- net RLED_RUN: now reaches D7.2 (A), R5.2
- net HOST_TX renamed RESET
- net RESET: now also TP7.1, U8.1, U8.2
- net MCU_CLK renamed HOST_SWCLK_RX
- net HOST_SWCLK_RX: now also TP11.1
- net MCU_DIO renamed HOST_SWDIO_TX
- net HOST_SWDIO_TX: now also TP10.1
- net MCU_RX renamed HOST_UART_RX
- net HOST_UART_RX: now also TP9.1
- net MCU_TX renamed HOST_UART_TX
- net HOST_UART_TX: now also TP8.1; no longer R19.1
- net QSPI_SCLK renamed QSPI_CLK
- removed net SHIELD: D3.1 (GND), J10.S1 (SHIELD), R12.1
- removed net VBUS: D3.4 (VCC), J10.A4 (VBUS), J10.A9 (VBUS), J10.B4 (VBUS), J10.B9 (VBUS)
- new net BOOTSEL: R7.2, TP6.1, U5.1, U5.2
- new net ROUT: C20.1, R12.2, Y1.3
- new net USBC_DN: D3.3 (I/O2), J10.5 (DN2), J10.7 (DN1), R25.2
- new net USBC_DP: D3.2 (I/O1), J10.6 (DP1), J10.8 (DP2), R24.2
- no-connect marks 22 -> 18
Other:
- note removed: "Alternative QSPI Flash with WSON footprint"
- note removed: "Boot source selection button"
- note removed: "Host protection"
- note removed: "LDO-based 3.3V power supply"
- note removed: "MCU JTAG connector"
- note removed: "MCU Reset line"
- note removed: "MCU UART connector"
- note removed: "Main MCU RP2040"
- note removed: "Main MCU crystal"
- note removed: "QSPI Flash with SOIC foorprint"
- note removed: "Status indication LEDs"
- note removed: "Target JTAG connector"
- note removed: "USB Type-C socket"
- note removed: "USB protection"
- company: (c) 2023 Andriy Golovnya -> (none)
- moved on the sheet: C10, C11, C14, C15, C16, C17, C18, C19, C2, C20, C3, C4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

Commit message: logo
Parts:
- TP10, TP11: footprint TestPoint:TestPoint_Pad_D1.0mm -> JLCPCB:TestPoint_Pad_1.0x1.0mm
- TP13, TP4, TP5, TP6, TP7, TP8, TP9: footprint TestPoint:TestPoint_Pad_D1.0mm -> JLCPCB:TestPoint_Pad_1.0x1.0mm; now left out of the parts list
Changed lines of the file:
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@@
 			)
 		)
-		(property "Footprint" "TestPoint:TestPoint_Pad_D1.0mm"
+		(property "Footprint" "JLCPCB:TestPoint_Pad_1.0x1.0mm"
 			(at 259.5881 116.84 0)
 			(effects
@@
 		(unit 1)
 		(exclude_from_sim no)
-		(in_bom yes)
+		(in_bom no)
 		(on_board yes)
 		(dnp no)
@@
 			)
 		)
-		(property "Footprint" "TestPoint:TestPoint_Pad_D1.0mm"
+		(property "Footprint" "JLCPCB:TestPoint_Pad_1.0x1.0mm"
 			(at 355.0919 45.72 0)
 			(effects
@@
 		(unit 1)
 		(exclude_from_sim no)
-		(in_bom yes)
+		(in_bom no)
 		(on_board yes)
 		(dnp no)
@@
 			)
 		)
-		(property "Footprint" "TestPoint:TestPoint_Pad_D1.0mm"
+		(property "Footprint" "JLCPCB:TestPoint_Pad_1.0x1.0mm"
 			(at 196.3419 91.44 0)
 			(effects
@@
 		(unit 1)
 		(exclude_from_sim no)
-		(in_bom yes)
+		(in_bom no)
 		(on_board yes)
 		(dnp no)
@@
 			)
 		)
-		(property "Footprint" "TestPoint:TestPoint_Pad_D1.0mm"
+		(property "Footprint" "JLCPCB:TestPoint_Pad_1.0x1.0mm"
 			(at 88.9 70.3581 0)
 			(effects
@@
 		(unit 1)
 		(exclude_from_sim no)
-		(in_bom yes)
+		(in_bom no)
 		(on_board yes)
 		(dnp no)
@@
 			)
 		)
-		(property "Footprint" "TestPoint:TestPoint_Pad_D1.0mm"
+		(property "Footprint" "JLCPCB:TestPoint_Pad_1.0x1.0mm"
 			(at 355.0919 43.18 0)
 			(effects
@@
 		(unit 1)
 		(exclude_from_sim no)
-		(in_bom yes)
+		(in_bom no)
 		(on_board yes)
 		(dnp no)
@@
 			)
 		)
-		(property "Footprint" "TestPoint:TestPoint_Pad_D1.0mm"
+		(property "Footprint" "JLCPCB:TestPoint_Pad_1.0x1.0mm"
 			(at 153.1619 77.47 0)
 			(effects
@@
 	)
 	(symbol
+		(lib_id "Graphic:Logo_Open_Hardware_Small")
+		(at 132.08 186.69 0)
+		(unit 1)
+		(exclude_from_sim yes)
+		(in_bom yes)
+		(on_board yes)
+		(dnp no)
+		(fields_autoplaced yes)
+		(property "Reference" "#SYM1"
+			(at 132.08 179.705 0)
+			(effects
+				(font
+					(size 1.27 1.27)
+				)
+				(hide yes)
+			)
+		)
+		(property "Value" "Logo_Open_Hardware_Small"
+			(at 132.08 192.405 0)
+			(effects
+				(font
+					(size 1.27 1.27)
+				)
+				(hide yes)
+			)
+		)
+		(property "Footprint" "Pixel:Logo B"
+			(at 132.08 186.69 0)
+			(effects
+				(font
+					(size 1.27 1.27)
+				)
+				(hide yes)
+			)
+		)
+		(property "Datasheet" "~"
+			(at 132.08 186.69 0)
+			(effects
+				(font
+					(size 1.27 1.27)
+				)
+				(hide yes)
+			)
+		)
+		(property "Description" "Open Hardware logo, small"
+			(at 132.08 186.69 0)
+			(effects
+				(font
+					(size 1.27 1.27)
+				)
+				(hide yes)
+			)
+		)
+		(instances
+			(project ""
+				(path "/9a38a81c-7302-494f-9784-2ab4342a0a1d"
+					(reference "#SYM1")
+					(unit 1)
+				)
+			)
+		)
+	)
+	(symbol
 		(lib_id "Device:R_Small")
 		(at 81.28 170.18 270)
@@
 		(unit 1)
 		(exclude_from_sim no)
-		(in_bom yes)
+		(in_bom no)
 		(on_board yes)
 		(dnp no)
@@
 			)
 		)
-		(property "Footprint" "TestPoint:TestPoint_Pad_D1.0mm"
+		(property "Footprint" "JLCPCB:TestPoint_Pad_1.0x1.0mm"
 			(at 219.2019 91.44 0)
 			(effects
@@
 			)
 		)
-		(property "Footprint" "TestPoint:TestPoint_Pad_D1.0mm"
+		(property "Footprint" "JLCPCB:TestPoint_Pad_1.0x1.0mm"
 			(at 259.5881 114.3 0)
 			(effects
@@
 		(unit 1)
 		(exclude_from_sim no)
-		(in_bom yes)
+		(in_bom no)
 		(on_board yes)
 		(dnp no)
@@
 			)
 		)
-		(property "Footprint" "TestPoint:TestPoint_Pad_D1.0mm"
+		(property "Footprint" "JLCPCB:TestPoint_Pad_1.0x1.0mm"
 			(at 302.26 30.9881 0)
 			(effects
